File: hardware/EurorackDualPitchQuantizerBack/EurorackDualPitchQuantizerBack.kicad_sch (KiCad schematic)
At the start: 41 parts, among them J1 Conn_01x04_Female, J10 Conn_01x02_Female, J2 Conn_01x12_Female, J3 Conn_02x05_Odd_Even, J4 Conn_01x02_Female, J5 MCP4725Breakout, J6 MCP4725Breakout, J7 Conn_01x12_Female, J8 Conn_01x02_Female, J9 Conn_01x01_Female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

Commit message: Got Rev 1.2 complete. It should be manufacturable and fit into eurorack standards.
Parts:
- removed J7: Conn_01x12_Female, Connector_PinSocket_2.54mm:PinSocket_1x12_P2.54mm_Vertical, symbol Connector:Conn_01x12_Female
- removed J9: Conn_01x01_Female, symbol Connector:Conn_01x01_Female
- removed U4, U5: 4021, Package_DIP:DIP-16_W7.62mm_Socket, symbol 4xxx:4021
- added J7: Conn_01x03_Female, Connector_PinHeader_2.54mm:PinHeader_1x03_P2.54mm_Vertical, symbol Connector:Conn_01x03_Female
- J1: footprint (none) -> Connector_PinSocket_2.54mm:PinSocket_1x04_P2.54mm_Vertical
- J10: footprint (none) -> Connector_PinHeader_2.54mm:PinHeader_1x02_P2.54mm_Vertical
- J8: footprint (none) -> Connector_PinSocket_2.54mm:PinSocket_1x02_P2.54mm_Vertical
Connections:
- net l1: now also J4.1 (Pin_1); no longer J2.12 (Pin_12)
- net l10: now also J2.5 (Pin_5); no longer J2.3 (Pin_3)
- net l11: now also J2.4 (Pin_4); no longer J2.2 (Pin_2)
- net l12: now also J2.3 (Pin_3); no longer J2.1 (Pin_1)
- net l13: now also J2.2 (Pin_2); no longer J4.1 (Pin_1)
- net l14: now also J2.1 (Pin_1); no longer J4.2 (Pin_2)
- net l2: now also J4.2 (Pin_2); no longer J2.11 (Pin_11)
- net l3: now also J2.12 (Pin_12); no longer J2.10 (Pin_10)
- net l4: now also J2.11 (Pin_11); no longer J2.9 (Pin_9)
- net l5: now also J2.10 (Pin_10); no longer J2.8 (Pin_8)
- net l6: now also J2.9 (Pin_9); no longer J2.7 (Pin_7)
- net l7: now also J2.8 (Pin_8); no longer J2.6 (Pin_6)
- net l8: now also J2.7 (Pin_7); no longer J2.5 (Pin_5)
- net l9: now also J2.6 (Pin_6); no longer J2.4 (Pin_4)
- net at A1.10 (D7): now also J7.3 (Pin_3)
- net at A1.11 (D8): now also J7.2 (Pin_2)
- net at A1.12 (D9): now also J7.1 (Pin_1)
- net at R18.2, U3.7: now also J8.1 (Pin_1); no longer J8.2 (Pin_2)
- net at R17.2, U3.1: now also J8.2 (Pin_2); no longer J8.1 (Pin_1)
- no-connect marks 30 -> 22
Other:
- company: (none) -> Ilmari Hirvonen
- title: (none) -> Dual Pitch Quantizer Back PCB
- moved on the sheet: J4
