File: hardware/EurorackDualPitchQuantizerFrontPanel/EurorackDualPitchQuantizerFrontPanel.kicad_sch (KiCad schematic)
At the start: 1 part, among them J1 Conn_01x01_Male

Commit message: Got Rev 1.2 complete. It should be manufacturable and fit into eurorack standards.
Other:
- company: (none) -> Ilmari Hirvonen
- title: (none) -> Dual Pitch Quantizer Front Panel
Changed lines of the file:
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@@
 (kicad_sch (version 20211123) (generator eeschema)
   (paper "A4")
+  (title_block
+    (title "Dual Pitch Quantizer Front Panel")
+    (date "2022-12-11")
+    (rev "1.2")
+    (company "Ilmari Hirvonen")
+    (comment 1 "License: CERN-OHL-S v2")
+  )
   (junction (at 149.225 98.425) (diameter 0) (color 0 0 0 0)
   )
